Commit message: Add dual-arm logic and related scripts/assets

File: assets/Xacro/panda_dual_arms.xacro (robot description, xacro)
@@ -4,7 +4,7 @@
   <xacro:arg name="arm_id_2" default="panda_right"/>
   <!-- Placement for each arm: xyz and rpy relative to world -->
-  <xacro:arg name="arm_1_xyz" default="0 0.5 0"/>
+  <xacro:arg name="arm_1_xyz" default="0 0.3 0"/>
   <xacro:arg name="arm_1_rpy" default="0 0 0"/>
-  <xacro:arg name="arm_2_xyz" default="0 -0.5 0"/>
+  <xacro:arg name="arm_2_xyz" default="0 -0.3 0"/>
   <xacro:arg name="arm_2_rpy" default="0 0 0"/>
   <material name="panda_white">

File: assets/urdf/panda/panda_dual_arms.urdf (robot description, URDF)
Before this commit: robot panda_dual_arms, 19 links, 18 joints
Joints:
- joint panda_left_base_joint: origin xyz=0 0.5 0 rpy=0 0 0 -> xyz=0 0.3 0 rpy=0 0 0
- joint panda_right_base_joint: origin xyz=0 -0.5 0 rpy=0 0 0 -> xyz=0 -0.3 0 rpy=0 0 0
